Commit message: Major Changes urdf/xacroandgazebo both launch files bridge.yaml file

File: mr_robot_description/urdf/mr_robot.xacro (robot description, xacro)
@@ -52,5 +52,17 @@
   </collision>
 </link>
- <!-- <link name="camera_link">
+<joint name="camera_joint" type="fixed">
+    <axis xyz="0 0.05 0"/>
+    <origin rpy="0 0 0" xyz="0.05 0 0.9"/>
+    <parent link="base_link"/>
+    <child link="camera_link"/>
+  </joint>
+<joint name="camera_optical_joint" type="fixed">
+    <parent link="camera_link"/>
+    <child link="camera_link_optical"/>
+    <origin xyz="0 0 0" rpy="${-pi/2} 0 ${-pi/2}"/>
+  </joint>
+<link name="camera_link_optical"></link>
+ <link name="camera_link">
     <collision>
       <origin rpy="0 0 0" xyz="0 0 0"/>
@@ -60,5 +72,5 @@
     </collision>
     <visual>
-      <origin rpy="0 0 0" xyz="0 0 0"/>
+      <origin rpy="0 0 0" xyz="0 0 0"/>     <!-- roll pitch and yaw in radians and xyz in meters-->
       <geometry>
         <box size="0.05 0.05 0.05"/>
@@ -71,12 +83,6 @@
       <inertia ixx="1e-6" ixy="0" ixz="0" iyy="1e-6" iyz="0" izz="1e-6"/>
     </inertial>
-  </link> -->
-  <!-- <joint name="camera_joint" type="fixed">
-    <axis xyz="0 1 0"/>
-    <origin rpy="0 0 0" xyz="0.05 0 0.9"/>
-    <parent link="link3"/>
-    <child link="camera_link"/>
-  </joint> -->
-<link name="Wheel_r_1">
+  </link>
+  <link name="Wheel_r_1">
   <inertial>
     <origin xyz="7.587052287765051e-07 -0.023812499999986303 5.494367044764359e-06" rpy="0 0 0"/>
