Commit message: changes

File: mr_robot_description/urdf/materials.xacro (robot description, xacro)
@@ -16,3 +16,6 @@
   <color rgba="0.0 1.0 0.0 1.0"/>
 </material>
+<material name="dark_blue">
+  <color rgba="0.0 0.0 0.75 1.0"/>
+</material>
 </robot>

File: mr_robot_description/urdf/mr_robot.xacro (robot description, xacro)
@@ -53,6 +53,6 @@
 </link>
 <joint name="camera_joint" type="fixed">
-    <axis xyz="0 0.05 0"/>
-    <origin rpy="0 0 0" xyz="0.05 0 0.9"/>
+    <axis xyz="0 0 0"/>
+    <origin rpy="0 0 0" xyz="0.27 0 0.14"/>
     <parent link="base_link"/>
     <child link="camera_link"/>
@@ -84,4 +84,30 @@
     </inertial>
   </link>
+  <joint name="depth_camera_joint" type="fixed">
+    <axis xyz="0 0 0" />
+    <origin xyz="0.27 0.1 0.14" rpy="0 0 0"/>
+    <parent link="base_link"/>
+    <child link="mr_robot/base_link/depth_camera"/>
+  </joint>
+  <link name="mr_robot/base_link/depth_camera">
+    <collision>
+      <origin xyz="0 0 0" rpy="0 0 0"/>
+      <geometry>
+    <box size="0.05 0.05 0.05"/>
+      </geometry>
+    </collision>
+    <visual>
+      <origin xyz="0 0 0" rpy="0 0 0"/>
+      <geometry>
+    <box size="0.05 0.05 0.05"/>
+      </geometry>
+      <material name="dark_blue"/>
+    </visual>
+    <inertial>
+      <mass value="1e-5" />
+      <origin xyz="0 0 0" rpy="0 0 0"/>
+      <inertia ixx="1e-6" ixy="0" ixz="0" iyy="1e-6" iyz="0" izz="1e-6" />
+    </inertial>
+  </link>
   <link name="Wheel_r_1">
   <inertial>
@@ -105,5 +131,5 @@
 </link>
 <joint name="imu_joint" type="fixed">
-  <origin xyz="0 0 0.2" rpy="0 0 0"/>
+  <origin xyz="0 0 0.18" rpy="0 0 0"/>
   <parent link="base_link"/>
   <child link="imu_link"/>
